File: otterworks_arrow.kicad_pcb (KiCad board)
At the start: 4 copper layers, 60 x 121 mm, 137 parts, among them U1 STM32F030C6Tx

Commit message: bottom side done
Parts:
- added C100: 100n, Capacitor_SMD:C_0603_1608Metric, B.Cu at (83.0, 125.0)
- added C101: 100n, Capacitor_SMD:C_0603_1608Metric, B.Cu at (75.0, 125.0)
- added C102: 100n, Capacitor_SMD:C_0603_1608Metric, B.Cu at (79.0, 133.0)
- added C103: 100n, Capacitor_SMD:C_0603_1608Metric, B.Cu at (83.0, 141.0)
- added C104: 100n, Capacitor_SMD:C_0603_1608Metric, B.Cu at (71.0, 101.0)
- added C105: 100n, Capacitor_SMD:C_0603_1608Metric, B.Cu at (87.0, 133.0)
- added C106: 100n, Capacitor_SMD:C_0603_1608Metric, B.Cu at (99.0, 53.0)
- added C107: 100n, Capacitor_SMD:C_0603_1608Metric, B.Cu at (75.0, 85.0)
- added C108: 100n, Capacitor_SMD:C_0603_1608Metric, B.Cu at (83.0, 109.0)
- added C109: 100n, Capacitor_SMD:C_0603_1608Metric, B.Cu at (83.0, 85.0)
- added C110: 100n, Capacitor_SMD:C_0603_1608Metric, B.Cu at (91.0, 53.0)
- added C111: 100n, Capacitor_SMD:C_0603_1608Metric, B.Cu at (91.0, 109.0)
- added C112: 100n, Capacitor_SMD:C_0603_1608Metric, B.Cu at (99.0, 109.0)
- added C113: 100n, Capacitor_SMD:C_0603_1608Metric, B.Cu at (75.0, 53.0)
- added C114: 100n, Capacitor_SMD:C_0603_1608Metric, B.Cu at (99.0, 45.0)
- added C115: 100n, Capacitor_SMD:C_0603_1608Metric, B.Cu at (67.0, 53.0)
- added C116: 100n, Capacitor_SMD:C_0603_1608Metric, B.Cu at (99.0, 61.0)
- added C117: 100n, Capacitor_SMD:C_0603_1608Metric, B.Cu at (59.0, 93.0)
- added C118: 100n, Capacitor_SMD:C_0603_1608Metric, B.Cu at (91.0, 85.0)
- added C119: 100n, Capacitor_SMD:C_0603_1608Metric, B.Cu at (91.0, 61.0)
- added C120: 100n, Capacitor_SMD:C_0603_1608Metric, B.Cu at (75.0, 61.0)
- added C121: 100n, Capacitor_SMD:C_0603_1608Metric, B.Cu at (99.0, 85.0)
- added C122: 100n, Capacitor_SMD:C_0603_1608Metric, B.Cu at (67.0, 109.0)
- added C123: 100n, Capacitor_SMD:C_0603_1608Metric, B.Cu at (87.0, 101.0)
- added C124: 100n, Capacitor_SMD:C_0603_1608Metric, B.Cu at (75.0, 109.0)
- added C125: 100n, Capacitor_SMD:C_0603_1608Metric, B.Cu at (103.0, 101.0)
- added C126: 100n, Capacitor_SMD:C_0603_1608Metric, B.Cu at (95.0, 101.0)
- added C127: 100n, Capacitor_SMD:C_0603_1608Metric, B.Cu at (83.0, 77.0)
- added C128: 100n, Capacitor_SMD:C_0603_1608Metric, B.Cu at (91.0, 77.0)
- added C129: 100n, Capacitor_SMD:C_0603_1608Metric, B.Cu at (99.0, 77.0)
- added C130: 100n, Capacitor_SMD:C_0603_1608Metric, B.Cu at (67.0, 85.0)
- added C131: 100n, Capacitor_SMD:C_0603_1608Metric, B.Cu at (83.0, 29.0)
- added C132: 100n, Capacitor_SMD:C_0603_1608Metric, B.Cu at (83.0, 53.0)
- added C133: 100n, Capacitor_SMD:C_0603_1608Metric, B.Cu at (67.0, 29.0)
- added C134: 100n, Capacitor_SMD:C_0603_1608Metric, B.Cu at (67.0, 61.0)
- added C135: 100n, Capacitor_SMD:C_0603_1608Metric, B.Cu at (75.0, 29.0)
- added C136: 100n, Capacitor_SMD:C_0603_1608Metric, B.Cu at (91.0, 29.0)
- added C69: 100n, Capacitor_SMD:C_0603_1608Metric, B.Cu at (79.0, 101.0)
- added C70: 100n, Capacitor_SMD:C_0603_1608Metric, B.Cu at (99.0, 69.0)
- added C71: 100n, Capacitor_SMD:C_0603_1608Metric, B.Cu at (75.0, 45.0)
- added C72: 100n, Capacitor_SMD:C_0603_1608Metric, B.Cu at (83.0, 45.0)
- added C73: 100n, Capacitor_SMD:C_0603_1608Metric, B.Cu at (67.0, 77.0)
- added C74: 100n, Capacitor_SMD:C_0603_1608Metric, B.Cu at (91.0, 45.0)
- added C75: 100n, Capacitor_SMD:C_0603_1608Metric, B.Cu at (75.0, 77.0)
- added C76: 100n, Capacitor_SMD:C_0603_1608Metric, B.Cu at (107.0, 93.0)
- added C77: 100n, Capacitor_SMD:C_0603_1608Metric, B.Cu at (83.0, 93.0)
- added C78: 100n, Capacitor_SMD:C_0603_1608Metric, B.Cu at (63.0, 101.0)
- added C79: 100n, Capacitor_SMD:C_0603_1608Metric, B.Cu at (99.0, 93.0)
- added C80: 100n, Capacitor_SMD:C_0603_1608Metric, B.Cu at (91.0, 93.0)
- added C81: 100n, Capacitor_SMD:C_0603_1608Metric, B.Cu at (91.0, 37.0)
- added C82: 100n, Capacitor_SMD:C_0603_1608Metric, B.Cu at (75.0, 37.0)
- added C83: 100n, Capacitor_SMD:C_0603_1608Metric, B.Cu at (67.0, 37.0)
- added C84: 100n, Capacitor_SMD:C_0603_1608Metric, B.Cu at (83.0, 37.0)
- added C85: 100n, Capacitor_SMD:C_0603_1608Metric, B.Cu at (83.0, 61.0)
- added C86: 100n, Capacitor_SMD:C_0603_1608Metric, B.Cu at (99.0, 29.0)
- added C87: 100n, Capacitor_SMD:C_0603_1608Metric, B.Cu at (67.0, 69.0)
- added C88: 100n, Capacitor_SMD:C_0603_1608Metric, B.Cu at (95.0, 117.0)
- added C89: 100n, Capacitor_SMD:C_0603_1608Metric, B.Cu at (87.0, 117.0)
- added C90: 100n, Capacitor_SMD:C_0603_1608Metric, B.Cu at (79.0, 117.0)
- added C91: 100n, Capacitor_SMD:C_0603_1608Metric, B.Cu at (71.0, 117.0)
- added C92: 100n, Capacitor_SMD:C_0603_1608Metric, B.Cu at (67.0, 93.0)
- added C93: 100n, Capacitor_SMD:C_0603_1608Metric, B.Cu at (75.0, 93.0)
- added C94: 100n, Capacitor_SMD:C_0603_1608Metric, B.Cu at (83.0, 69.0)
- added C95: 100n, Capacitor_SMD:C_0603_1608Metric, B.Cu at (67.0, 45.0)
- added C96: 100n, Capacitor_SMD:C_0603_1608Metric, B.Cu at (75.0, 69.0)
- added C97: 100n, Capacitor_SMD:C_0603_1608Metric, B.Cu at (99.0, 37.0)
- added C98: 100n, Capacitor_SMD:C_0603_1608Metric, B.Cu at (91.0, 69.0)
- added C99: 100n, Capacitor_SMD:C_0603_1608Metric, B.Cu at (91.0, 125.0)
- added D100: WS2812B-2020, LED_SMD:LED_WS2812B_PLCC4_5.0x5.0mm_P3.2mm, B.Cu at (83.0, 121.0)
- added D101: WS2812B-2020, LED_SMD:LED_WS2812B_PLCC4_5.0x5.0mm_P3.2mm, B.Cu at (75.0, 121.0)
- added D102: WS2812B-2020, LED_SMD:LED_WS2812B_PLCC4_5.0x5.0mm_P3.2mm, B.Cu at (79.0, 129.0)
- added D103: WS2812B-2020, LED_SMD:LED_WS2812B_PLCC4_5.0x5.0mm_P3.2mm, B.Cu at (83.0, 137.0)
- added D104: WS2812B-2020, LED_SMD:LED_WS2812B_PLCC4_5.0x5.0mm_P3.2mm, B.Cu at (71.0, 97.0)
- added D105: WS2812B-2020, LED_SMD:LED_WS2812B_PLCC4_5.0x5.0mm_P3.2mm, B.Cu at (87.0, 129.0)
- added D106: WS2812B-2020, LED_SMD:LED_WS2812B_PLCC4_5.0x5.0mm_P3.2mm, B.Cu at (99.0, 49.0)
- added D107: WS2812B-2020, LED_SMD:LED_WS2812B_PLCC4_5.0x5.0mm_P3.2mm, B.Cu at (75.0, 81.0)
- added D108: WS2812B-2020, LED_SMD:LED_WS2812B_PLCC4_5.0x5.0mm_P3.2mm, B.Cu at (83.0, 105.0)
- added D109: WS2812B-2020, LED_SMD:LED_WS2812B_PLCC4_5.0x5.0mm_P3.2mm, B.Cu at (83.0, 81.0)
- added D110: WS2812B-2020, LED_SMD:LED_WS2812B_PLCC4_5.0x5.0mm_P3.2mm, B.Cu at (91.0, 49.0)
- added D111: WS2812B-2020, LED_SMD:LED_WS2812B_PLCC4_5.0x5.0mm_P3.2mm, B.Cu at (91.0, 105.0)
- added D112: WS2812B-2020, LED_SMD:LED_WS2812B_PLCC4_5.0x5.0mm_P3.2mm, B.Cu at (99.0, 105.0)
- added D113: WS2812B-2020, LED_SMD:LED_WS2812B_PLCC4_5.0x5.0mm_P3.2mm, B.Cu at (75.0, 49.0)
- added D114: WS2812B-2020, LED_SMD:LED_WS2812B_PLCC4_5.0x5.0mm_P3.2mm, B.Cu at (99.0, 41.0)
- added D115: WS2812B-2020, LED_SMD:LED_WS2812B_PLCC4_5.0x5.0mm_P3.2mm, B.Cu at (67.0, 49.0)
- added D116: WS2812B-2020, LED_SMD:LED_WS2812B_PLCC4_5.0x5.0mm_P3.2mm, B.Cu at (99.0, 57.0)
- added D117: WS2812B-2020, LED_SMD:LED_WS2812B_PLCC4_5.0x5.0mm_P3.2mm, B.Cu at (59.0, 89.0)
- added D118: WS2812B-2020, LED_SMD:LED_WS2812B_PLCC4_5.0x5.0mm_P3.2mm, B.Cu at (91.0, 81.0)
- added D119: WS2812B-2020, LED_SMD:LED_WS2812B_PLCC4_5.0x5.0mm_P3.2mm, B.Cu at (91.0, 57.0)
- added D120: WS2812B-2020, LED_SMD:LED_WS2812B_PLCC4_5.0x5.0mm_P3.2mm, B.Cu at (75.0, 57.0)
- added D121: WS2812B-2020, LED_SMD:LED_WS2812B_PLCC4_5.0x5.0mm_P3.2mm, B.Cu at (99.0, 81.0)
- added D122: WS2812B-2020, LED_SMD:LED_WS2812B_PLCC4_5.0x5.0mm_P3.2mm, B.Cu at (67.0, 105.0)
- added D123: WS2812B-2020, LED_SMD:LED_WS2812B_PLCC4_5.0x5.0mm_P3.2mm, B.Cu at (87.0, 97.0)
- added D124: WS2812B-2020, LED_SMD:LED_WS2812B_PLCC4_5.0x5.0mm_P3.2mm, B.Cu at (75.0, 105.0)
- added D125: WS2812B-2020, LED_SMD:LED_WS2812B_PLCC4_5.0x5.0mm_P3.2mm, B.Cu at (103.0, 97.0)
- added D126: WS2812B-2020, LED_SMD:LED_WS2812B_PLCC4_5.0x5.0mm_P3.2mm, B.Cu at (95.0, 97.0)
- added D127: WS2812B-2020, LED_SMD:LED_WS2812B_PLCC4_5.0x5.0mm_P3.2mm, B.Cu at (83.0, 73.0)
- added D128: WS2812B-2020, LED_SMD:LED_WS2812B_PLCC4_5.0x5.0mm_P3.2mm, B.Cu at (91.0, 73.0)
- added D129: WS2812B-2020, LED_SMD:LED_WS2812B_PLCC4_5.0x5.0mm_P3.2mm, B.Cu at (99.0, 73.0)
- added D130: WS2812B-2020, LED_SMD:LED_WS2812B_PLCC4_5.0x5.0mm_P3.2mm, B.Cu at (67.0, 81.0)
- added D131: WS2812B-2020, LED_SMD:LED_WS2812B_PLCC4_5.0x5.0mm_P3.2mm, B.Cu at (83.0, 25.0)
- added D132: WS2812B-2020, LED_SMD:LED_WS2812B_PLCC4_5.0x5.0mm_P3.2mm, B.Cu at (83.0, 49.0)
- added D133: WS2812B-2020, LED_SMD:LED_WS2812B_PLCC4_5.0x5.0mm_P3.2mm, B.Cu at (67.0, 25.0)
- added D134: WS2812B-2020, LED_SMD:LED_WS2812B_PLCC4_5.0x5.0mm_P3.2mm, B.Cu at (67.0, 57.0)
- added D135: WS2812B-2020, LED_SMD:LED_WS2812B_PLCC4_5.0x5.0mm_P3.2mm, B.Cu at (75.0, 25.0)
- added D136: WS2812B-2020, LED_SMD:LED_WS2812B_PLCC4_5.0x5.0mm_P3.2mm, B.Cu at (91.0, 25.0)
- added D69: WS2812B-2020, LED_SMD:LED_WS2812B_PLCC4_5.0x5.0mm_P3.2mm, B.Cu at (79.0, 97.0)
- added D70: WS2812B-2020, LED_SMD:LED_WS2812B_PLCC4_5.0x5.0mm_P3.2mm, B.Cu at (99.0, 65.0)
- added D71: WS2812B-2020, LED_SMD:LED_WS2812B_PLCC4_5.0x5.0mm_P3.2mm, B.Cu at (75.0, 41.0)
- added D72: WS2812B-2020, LED_SMD:LED_WS2812B_PLCC4_5.0x5.0mm_P3.2mm, B.Cu at (83.0, 41.0)
- added D73: WS2812B-2020, LED_SMD:LED_WS2812B_PLCC4_5.0x5.0mm_P3.2mm, B.Cu at (67.0, 73.0)
- added D74: WS2812B-2020, LED_SMD:LED_WS2812B_PLCC4_5.0x5.0mm_P3.2mm, B.Cu at (91.0, 41.0)
- added D75: WS2812B-2020, LED_SMD:LED_WS2812B_PLCC4_5.0x5.0mm_P3.2mm, B.Cu at (75.0, 73.0)
- added D76: WS2812B-2020, LED_SMD:LED_WS2812B_PLCC4_5.0x5.0mm_P3.2mm, B.Cu at (107.0, 89.0)
- added D77: WS2812B-2020, LED_SMD:LED_WS2812B_PLCC4_5.0x5.0mm_P3.2mm, B.Cu at (83.0, 89.0)
- added D78: WS2812B-2020, LED_SMD:LED_WS2812B_PLCC4_5.0x5.0mm_P3.2mm, B.Cu at (63.0, 97.0)
- added D79: WS2812B-2020, LED_SMD:LED_WS2812B_PLCC4_5.0x5.0mm_P3.2mm, B.Cu at (99.0, 89.0)
- added D80: WS2812B-2020, LED_SMD:LED_WS2812B_PLCC4_5.0x5.0mm_P3.2mm, B.Cu at (91.0, 89.0)
- added D81: WS2812B-2020, LED_SMD:LED_WS2812B_PLCC4_5.0x5.0mm_P3.2mm, B.Cu at (91.0, 33.0)
- added D82: WS2812B-2020, LED_SMD:LED_WS2812B_PLCC4_5.0x5.0mm_P3.2mm, B.Cu at (75.0, 33.0)
- added D83: WS2812B-2020, LED_SMD:LED_WS2812B_PLCC4_5.0x5.0mm_P3.2mm, B.Cu at (67.0, 33.0)
- added D84: WS2812B-2020, LED_SMD:LED_WS2812B_PLCC4_5.0x5.0mm_P3.2mm, B.Cu at (83.0, 33.0)
- added D85: WS2812B-2020, LED_SMD:LED_WS2812B_PLCC4_5.0x5.0mm_P3.2mm, B.Cu at (83.0, 57.0)
- added D86: WS2812B-2020, LED_SMD:LED_WS2812B_PLCC4_5.0x5.0mm_P3.2mm, B.Cu at (99.0, 25.0)
- added D87: WS2812B-2020, LED_SMD:LED_WS2812B_PLCC4_5.0x5.0mm_P3.2mm, B.Cu at (67.0, 65.0)
- added D88: WS2812B-2020, LED_SMD:LED_WS2812B_PLCC4_5.0x5.0mm_P3.2mm, B.Cu at (95.0, 113.0)
- added D89: WS2812B-2020, LED_SMD:LED_WS2812B_PLCC4_5.0x5.0mm_P3.2mm, B.Cu at (87.0, 113.0)
- added D90: WS2812B-2020, LED_SMD:LED_WS2812B_PLCC4_5.0x5.0mm_P3.2mm, B.Cu at (79.0, 113.0)
- added D91: WS2812B-2020, LED_SMD:LED_WS2812B_PLCC4_5.0x5.0mm_P3.2mm, B.Cu at (71.0, 113.0)
- added D92: WS2812B-2020, LED_SMD:LED_WS2812B_PLCC4_5.0x5.0mm_P3.2mm, B.Cu at (67.0, 89.0)
- added D93: WS2812B-2020, LED_SMD:LED_WS2812B_PLCC4_5.0x5.0mm_P3.2mm, B.Cu at (75.0, 89.0)
- added D94: WS2812B-2020, LED_SMD:LED_WS2812B_PLCC4_5.0x5.0mm_P3.2mm, B.Cu at (83.0, 65.0)
- added D95: WS2812B-2020, LED_SMD:LED_WS2812B_PLCC4_5.0x5.0mm_P3.2mm, B.Cu at (67.0, 41.0)
- added D96: WS2812B-2020, LED_SMD:LED_WS2812B_PLCC4_5.0x5.0mm_P3.2mm, B.Cu at (75.0, 65.0)
- added D97: WS2812B-2020, LED_SMD:LED_WS2812B_PLCC4_5.0x5.0mm_P3.2mm, B.Cu at (99.0, 33.0)
- added D98: WS2812B-2020, LED_SMD:LED_WS2812B_PLCC4_5.0x5.0mm_P3.2mm, B.Cu at (91.0, 65.0)
- added D99: WS2812B-2020, LED_SMD:LED_WS2812B_PLCC4_5.0x5.0mm_P3.2mm, B.Cu at (91.0, 121.0)
- moved C1 48.8 mm to (83.0, 141.0)
- moved C10 48.8 mm to (71.0, 117.0)
- moved C11 48.8 mm to (99.0, 109.0)
- moved C12 48.8 mm to (91.0, 109.0)
- moved C13 48.8 mm to (83.0, 109.0)
- moved C14 48.8 mm to (75.0, 109.0)
- moved C15 48.8 mm to (67.0, 109.0)
- moved C16 48.8 mm to (103.0, 101.0)
- moved C17 48.8 mm to (95.0, 101.0)
- moved C18 48.8 mm to (87.0, 101.0)
- moved C19 48.8 mm to (79.0, 101.0)
- moved C2 48.8 mm to (87.0, 133.0)
- moved C20 48.8 mm to (71.0, 101.0)
- moved C21 48.8 mm to (63.0, 101.0)
- moved C22 48.8 mm to (107.0, 93.0)
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Connections:
- U1 pad 29: unconnected-(U1-PA8-Pad29) -> /leds1/DIN
Routing:
- net GND: track 274.0 -> 3076.2 mm, vias 68 -> 269
- net +5V: track 497.3 -> 2857.0 mm, vias 68 -> 269
- net /leds1/ws2812_21/DOUT: track 0.00 -> 52.8 mm
- net /leds1/ws2812_28/DOUT: track 0.00 -> 48.8 mm
- net /leds1/ws2812_15/DOUT: track 0.00 -> 44.9 mm
- net /leds1/ws2812_58/DOUT: track 0.00 -> 40.9 mm
- net /leds1/ws2812_63/DOUT: track 0.00 -> 40.8 mm
- net /leds1/ws2812_48/DOUT: track 0.00 -> 40.8 mm
- net /leds1/ws2812_38/DOUT: track 0.00 -> 40.8 mm
- net /leds1/ws2812_53/DOUT: track 0.00 -> 40.8 mm
- net /leds1/ws2812_43/DOUT: track 0.00 -> 40.8 mm
- net /leds1/ws2812_33/DOUT: track 0.00 -> 40.7 mm
- net /leds1/ws2812_10/DOUT: track 0.00 -> 36.9 mm
- net /leds1/ws2812_6/DOUT: track 0.00 -> 28.9 mm
- net /leds1/ws2812_3/DOUT: track 0.00 -> 20.9 mm
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Other:
- outline, holes or cut-outs redrawn

Commit message: bosh IMU addded
Parts:
- added C137: 470n, Capacitor_SMD:C_0603_1608Metric, F.Cu at (100.8, 156.3)
- added C138: 100n, Capacitor_SMD:C_0603_1608Metric, F.Cu at (97.8, 156.3)
- added C139: 1u, Capacitor_SMD:C_0603_1608Metric, F.Cu at (97.8, 157.9)
- added C140: 100n, Capacitor_SMD:C_0603_1608Metric, F.Cu at (102.0, 153.7)
- added U2: BHI160B, LGA24_3x3:LGA-24_3x3mm, F.Cu at (99.3, 153.5)

Commit message: wip
Parts:
- removed U1: STM32F030C6Tx, Package_QFP:LQFP-48_7x7mm_P0.5mm
- added C141: 100n, Capacitor_SMD:C_0603_1608Metric, F.Cu at (47.4, 153.8)
- added C142: 100n, Capacitor_SMD:C_0603_1608Metric, F.Cu at (47.4, 156.3)
- added C143: 100n, Capacitor_SMD:C_0603_1608Metric, F.Cu at (47.4, 158.8)
- added C144: 100n, Capacitor_SMD:C_0603_1608Metric, F.Cu at (47.4, 161.4)
- added FB1: ferrite, Inductor_SMD:L_0603_1608Metric, F.Cu at (47.4, 163.9)
- added J1: PROG, Connector_PinHeader_2.54mm:PinHeader_1x06_P2.54mm_Vertical, F.Cu at (94.1, 146.9)
- added R1: 0, Resistor_SMD:R_0603_1608Metric, F.Cu at (47.4, 166.4)
- added R10: 0, Resistor_SMD:R_0603_1608Metric, F.Cu at (58.6, 149.5)
- added R11: 0, Resistor_SMD:R_0603_1608Metric, F.Cu at (58.6, 152.0)
- added R12: 0, Resistor_SMD:R_0603_1608Metric, F.Cu at (58.6, 154.5)
- added R13: 10k, Resistor_SMD:R_0603_1608Metric, F.Cu at (58.6, 157.0)
- added R14: 10k, Resistor_SMD:R_0603_1608Metric, F.Cu at (58.6, 159.5)
- added R2: 10k, Resistor_SMD:R_0603_1608Metric, F.Cu at (47.4, 168.9)
- added R3: 10k, Resistor_SMD:R_0603_1608Metric, F.Cu at (54.6, 149.5)
- added R4: 100, Resistor_SMD:R_0603_1608Metric, F.Cu at (54.6, 152.0)
- added R5: 100, Resistor_SMD:R_0603_1608Metric, F.Cu at (54.6, 154.5)
- added R6: 100, Resistor_SMD:R_0603_1608Metric, F.Cu at (54.6, 157.0)
- added R7: 100, Resistor_SMD:R_0603_1608Metric, F.Cu at (54.6, 159.5)
- added R8: 2.2k, Resistor_SMD:R_0603_1608Metric, F.Cu at (54.6, 162.0)
- added R9: 2.2k, Resistor_SMD:R_0603_1608Metric, F.Cu at (54.6, 164.5)
- added SW1: SW_Push, Button_Switch_SMD:SW_Push_1P1T_NO_CK_KSC7xxJ, F.Cu at (67.5, 148.3)
- added TP0: TestPoint, TestPoint:TestPoint_Pad_D1.0mm, F.Cu at (111.1, 158.7)
- added TP1: TestPoint, TestPoint:TestPoint_Pad_D1.0mm, F.Cu at (111.1, 161.8)
- added TP2: TestPoint, TestPoint:TestPoint_Pad_D1.0mm, F.Cu at (111.1, 164.8)
- added TP3: TestPoint, TestPoint:TestPoint_Pad_D1.0mm, F.Cu at (114.2, 158.7)
- added TP4: TestPoint, TestPoint:TestPoint_Pad_D1.0mm, F.Cu at (114.2, 161.8)
- added TP5: TestPoint, TestPoint:TestPoint_Pad_D1.0mm, F.Cu at (114.2, 164.8)
- added TP6: TestPoint, TestPoint:TestPoint_Pad_D1.0mm, F.Cu at (117.2, 158.7)
- added TP7: TestPoint, TestPoint:TestPoint_Pad_D1.0mm, F.Cu at (117.2, 161.8)
- added TP8: TestPoint, TestPoint:TestPoint_Pad_D1.0mm, F.Cu at (117.2, 164.8)
- added U3: STM32F030K6Tx, Package_QFP:LQFP-32_7x7mm_P0.8mm, F.Cu at (80.7, 149.0)
- moved U2 9.83 mm to (89.6, 152.3)
- moved C137 9.83 mm to (91.1, 155.1)
- moved C138 9.83 mm to (88.0, 155.1)
- moved C139 9.83 mm to (88.0, 156.6)
- moved C140 9.83 mm to (92.2, 152.4)
Connections:
- U2 pad 12: unconnected-(U2-INT-Pad12) -> I2C1_INT
- U2 pad 23: unconnected-(U2-SCK-Pad23) -> I2C1_SCL
- U2 pad 24: unconnected-(U2-SDA-Pad24) -> I2C1_SDA

Commit message: wip
Parts:
- added C146: 100n, Capacitor_SMD:C_0603_1608Metric, F.Cu at (107.5, 163.0)
- added C147: 100n, Capacitor_SMD:C_0603_1608Metric, F.Cu at (100.2, 163.1)
- added C148: 100n, Capacitor_SMD:C_0603_1608Metric, F.Cu at (58.7, 163.2)
- added D137: BPW34, OptoDevice:Osram_DIL2_4.3x4.65mm_P5.08mm, F.Cu at (69.3, 158.4)
- added FB2: ferrite, Inductor_SMD:L_0603_1608Metric, F.Cu at (91.9, 156.6)
- added H1: MountingHole_Pad, MountingHole:MountingHole_3.2mm_M3_Pad, F.Cu at (47.2, 150.8)
- added H2: MountingHole_Pad, MountingHole:MountingHole_3.2mm_M3_Pad, F.Cu at (112.8, 150.0)
- added H3: MountingHole, MountingHole:MountingHole_6mm, F.Cu at (61.0, 155.0)
- added H4: MountingHole, MountingHole:MountingHole_6mm, F.Cu at (99.0, 155.0)
- added P1: USB_C_Plug_USB2.0, Connector_USB:USB_C_Receptacle_HRO_TYPE-C-31-M-12, F.Cu at (113.6, 159.4)
- added Q1: MMBT2484LT1G, Package_TO_SOT_SMD:SOT-23, F.Cu at (64.5, 163.0)
- added R15: 5.1k, Resistor_SMD:R_0603_1608Metric, F.Cu at (107.8, 152.6)
- added R16: 5.1k, Resistor_SMD:R_0603_1608Metric, F.Cu at (106.3, 152.6)
- added R17: 0, Resistor_SMD:R_0603_1608Metric, F.Cu at (105.0, 160.3)
- added R18: 33k, Resistor_SMD:R_0603_1608Metric, F.Cu at (84.3, 148.0)
- added R19: 10k, Resistor_SMD:R_0603_1608Metric, F.Cu at (84.3, 149.8)
- added R20: 10, Resistor_SMD:R_0603_1608Metric, F.Cu at (68.3, 155.6)
- added R21: 33k, Resistor_SMD:R_0603_1608Metric, F.Cu at (60.2, 163.2)
- added R22: 10k, Resistor_SMD:R_0603_1608Metric, F.Cu at (61.7, 163.2)
- added R23: 10k, Resistor_SMD:R_0603_1608Metric, F.Cu at (107.5, 159.7)
- added U1: ADP7142AUJZ-3.3, Package_TO_SOT_SMD:TSOT-23-5, F.Cu at (104.5, 163.0)
- moved TP8 49.2 mm to (72.9, 143.4)
- moved TP7 44.6 mm to (76.3, 143.9)
- moved TP6 40.5 mm to (79.5, 143.9)
- moved FB1 39.0 mm to (84.4, 151.5), turned to 180 degrees
- moved C143 36.2 mm to (83.5, 156.2)
- moved C141 36.1 mm to (83.5, 153.0)
- moved TP2 36.1 mm to (80.3, 146.2)
- moved R2 35.1 mm to (80.9, 158.4), turned to 90 degrees
- moved TP1 32.8 mm to (81.3, 148.2)
- moved TP0 32.0 mm to (82.3, 144.9)
- moved R8 31.0 mm to (85.5, 159.4), turned to -90 degrees
- moved R1 30.5 mm to (70.9, 147.1), turned to 180 degrees
- moved R3 30.4 mm to (84.5, 154.7), turned to 180 degrees
- moved R9 29.7 mm to (83.8, 159.3), turned to -90 degrees
- moved TP4 28.1 mm to (88.9, 149.5)
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Connections:
- net +3.3VA renamed Net-(U2-VDD)
- net Net-(U3-PA3) renamed /IN_SWITCH
- R9 pad 2: I2C1_SCL -> I2C1_SDA
- U3 pad 10: unconnected-(U3-PA4-Pad10) -> /IN_ADC_SUPPLY
- U3 pad 11: unconnected-(U3-PA5-Pad11) -> /IN_AMB_LIGHT
Routing:
- net I2C1_SCL: track 0.00 -> 36.5 mm, vias 0 -> 2
- net I2C1_SDA: track 0.00 -> 35.5 mm
- net I2C1_INT: track 0.00 -> 30.4 mm, vias 0 -> 2
- net Net-(U3-VDDA): track 0.00 -> 23.4 mm
- net GND: track 3076.2 -> 3097.1 mm, vias 269 -> 283
- net PROG_TX: track 0.00 -> 15.7 mm, vias 0 -> 2
- net PROG_BOOT0: track 0.00 -> 15.3 mm
- net +3.3V: track 0.00 -> 15.2 mm, vias 0 -> 5
- net +5V: track 2857.0 -> 2871.6 mm, vias 269 -> 273
- net Net-(J1-Pin_2): track 0.00 -> 13.4 mm
- net Net-(J1-Pin_4): track 0.00 -> 12.4 mm, vias 0 -> 1
- net PROG_RX: track 0.00 -> 11.6 mm
- net Net-(P1-CC): track 0.00 -> 9.22 mm
- net Net-(J1-Pin_6): track 0.00 -> 7.06 mm
- net Net-(P1-VCONN): track 0.00 -> 6.80 mm
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- added copper zone on In2.Cu, net +3.3V
- added copper zone on B.Cu, net GND
- added copper zone on F.Cu, net GND
Other:
- board size 60 x 121 mm -> 74 x 146 mm
