File: ws2812.kicad_sch (KiCad schematic)
At the start: 2 parts

Commit message: wip
Parts:
- renumbered C68 to C81, D1 to D81
Changed lines of the file:
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@@
 		(dnp no)
 		(fields_autoplaced yes)
-		(property "Reference" "C68"
+		(property "Reference" "C81"
 			(at 139.7 85.0962 0)
 			(effects
@@
 		(dnp no)
 		(fields_autoplaced yes)
-		(property "Reference" "#PWR01"
+		(property "Reference" "#PWR0241"
 			(at 133.35 85.09 0)
 			(effects
@@
 		(on_board yes)
 		(dnp no)
-		(property "Reference" "D1"
+		(property "Reference" "D81"
 			(at 137.16 105.156 0)
 			(effects
@@
 		(on_board yes)
 		(dnp no)
-		(property "Reference" "#PWR03"
+		(property "Reference" "#PWR0243"
 			(at 137.16 95.25 0)
 			(effects
@@
 		(dnp no)
 		(fields_autoplaced yes)
-		(property "Reference" "#PWR02"
+		(property "Reference" "#PWR0242"
 			(at 133.35 111.76 0)
 			(effects
